Commit message: metro urdf

File: metro_sim/urdf/metro.urdf (robot description, URDF)
Before this commit: robot metro, 11 links, 10 joints
Joints:
- joint base_to_back_chassis: axis (none) -> 1 0 0; limit (none) -> lower=-1.57 upper=1.57 effort=0.0 velocity=0.5; type fixed -> revolute
- joint base_to_bl_arm: origin xyz=${arm_x_offset} ${(chassis_width/2)+(arm_width/2)+safe_gap} -${arm_z_offset} -> xyz=${arm_x_offset} ${(chassis_width/2)+(arm_width/2)+safe_gap} -${arm_z_offset} rpy=0 ${-arm_angle} 0
- joint base_to_br_arm: origin xyz=${arm_x_offset} ${-((chassis_width/2)+(arm_width/2)+safe_gap)} -${arm_z_offset} -> xyz=${arm_x_offset} ${-((chassis_width/2)+(arm_width/2)+safe_gap)} -${arm_z_offset} rpy=0 ${-arm_angle} 0
- joint base_to_fl_arm: origin xyz=${-arm_x_offset} ${(chassis_width/2)+(arm_width/2)+safe_gap} -${arm_z_offset} -> xyz=${-arm_x_offset} ${(chassis_width/2)+(arm_width/2)+safe_gap} -${arm_z_offset} rpy=0 ${arm_angle} 0
- joint base_to_fr_arm: origin xyz=${-arm_x_offset} ${-((chassis_width/2)+(arm_width/2)+safe_gap)} -${arm_z_offset} -> xyz=${-arm_x_offset} ${-((chassis_width/2)+(arm_width/2)+safe_gap)} -${arm_z_offset} rpy=0 ${arm_angle} 0
