Commit message: passive joint

File: metro_sim/urdf/metro_ss.urdf (robot description, URDF)
Before this commit: robot metro_ss, 10 links, 9 joints
Links:
- link inertial_link: mass 46.034 -> 25
Joints:
- joint base_to_back_chassis: axis (none) -> 1 0 0; limit (none) -> lower=-2.5 upper=2.5 effort=0.0 velocity=0.5; type fixed -> revolute
