Commit message: upload

File: husky/husky_description/urdf/decorations.urdf.xacro (robot description, xacro)
@@ -22,4 +22,11 @@
 -->
 <robot name="husky_decorations" xmlns:xacro="http://ros.org/wiki/xacro">
+  <material name="dark_grey"><color rgba="0.2 0.2 0.2 1.0" /></material>
+  <material name="medium_grey"><color rgba="0.6 0.6 0.6 1.0" /></material>
+  <material name="light_grey"><color rgba="0.8 0.8 0.8 1.0" /></material>
+  <material name="yellow"><color rgba="0.8 0.8 0.0 1.0" /></material>
+  <material name="black"><color rgba="0.15 0.15 0.15 1.0" /></material>
+  <material name="white"><color rgba="1.0 1.0 1.0 1.0" /></material>
+  <material name="red"><color rgba="1.0 0.0 0.0 1.0" /></material>
   <xacro:macro name="husky_decorate">
     <xacro:property name="husky_front_bumper_extend" value="$(optenv HUSKY_FRONT_BUMPER_EXTEND 0)" />

File: husky/husky_description/urdf/husky.urdf.xacro (robot description, xacro)
@@ -25,17 +25,16 @@
   <xacro:arg name="laser_xyz" default="$(optenv HUSKY_LMS1XX_XYZ 0.2206 0.0 0.00635)" />
   <xacro:arg name="laser_rpy" default="$(optenv HUSKY_LMS1XX_RPY 0.0 0.0 0.0)" />
-  <xacro:arg name="kinect_enabled" default="false" />
-  <xacro:arg name="kinect_xyz" default="$(optenv HUSKY_KINECT_XYZ 0 0 0)" />
-  <xacro:arg name="kinect_rpy" default="$(optenv HUSKY_KINECT_RPY 0 0.18 3.14)" />
+  <xacro:arg name="realsense_enabled" default="false" />
+  <xacro:arg name="realsense_xyz" default="$(optenv HUSKY_REALSENSE_XYZ 0 0 0)" />
+  <xacro:arg name="realsense_rpy" default="$(optenv HUSKY_REALSENSE_RPY 0 0 0)" />
+  <xacro:arg name="realsense_mount" default="$(optenv HUSKY_REALSENSE_MOUNT_FRAME sensor_arch_mount_link)" />
   <xacro:property name="husky_front_bumper_extend" value="$(optenv HUSKY_FRONT_BUMPER_EXTEND 0)" />
   <xacro:property name="husky_rear_bumper_extend" value="$(optenv HUSKY_REAR_BUMPER_EXTEND 0)" />
   <xacro:arg name="robot_namespace" default="/" />
   <xacro:arg name="urdf_extras" default="empty.urdf" />
-  <xacro:arg name="gpu" default="false"/>
-  <xacro:property name="gpu" value="$(arg gpu)" />
   <!-- Included URDF/XACRO Files -->
   <xacro:include filename="$(find husky_description)/urdf/decorations.urdf.xacro" />
   <xacro:include filename="$(find husky_description)/urdf/wheel.urdf.xacro" />
-  <xacro:include filename="$(find husky_description)/urdf/accessories/kinect_camera.urdf.xacro"/>
+  <xacro:include filename="$(find husky_description)/urdf/accessories/intel_realsense.urdf.xacro"/>
   <xacro:include filename="$(find husky_description)/urdf/accessories/sick_lms1xx_mount.urdf.xacro"/>
   <xacro:include filename="$(find husky_description)/urdf/accessories/sensor_arch.urdf.xacro"/>
@@ -80,5 +79,5 @@
     <child link="base_footprint" />
   </joint>
-  <!-- Interial link stores the robot's inertial information -->
+  <!-- Inertial link stores the robot's inertial information -->
   <link name="inertial_link">
     <inertial>
@@ -97,5 +96,4 @@
   <link name="imu_link"/>
   <joint name="imu_joint" type="fixed">
-    <!-- default: <origin xyz="$(optenv HUSKY_IMU_XYZ 0.19 0 0.149)" rpy="$(optenv HUSKY_IMU_RPY 0 -1.5708 3.1416)" /> -->
     <origin xyz="$(optenv HUSKY_IMU_XYZ 0.19 0 0.149)" rpy="$(optenv HUSKY_IMU_RPY 0 -1.5708 3.1416)" />
     <parent link="base_link" />
@@ -127,20 +125,25 @@
     </joint>
   </xacro:if>
-  <xacro:if value="$(arg kinect_enabled)">
+  <!--
+    top sensor arch; include this if we have realsense enabled
+    keep this as a property to make it easier to add multiple conditions, should we need
+    the top bar for any additional sensors in the future
+  -->
+  <xacro:property name="topbar_needed_realsense" value="$(arg realsense_enabled)" />
+  <xacro:if value="${topbar_needed_realsense}">
     <xacro:sensor_arch prefix="" parent="top_plate_link">
       <origin xyz="-0.35 0 0.51" rpy="0 0 -3.14"/>
     </xacro:sensor_arch>
-    <joint name="kinect_frame_joint" type="fixed">
-      <origin xyz="$(arg kinect_xyz)" rpy="$(arg kinect_rpy)" />
-      <parent link="sensor_arch_mount_link"/>
-      <child link="camera_link"/>
+  </xacro:if>
+  <!-- add the intel realsense to the topbar if needed -->
+  <xacro:if value="$(arg realsense_enabled)">
+    <link name="realsense_mountpoint"/>
+    <joint name="realsense_mountpoint_joint" type="fixed">
+      <origin xyz="0 0 0" rpy="0 0 -3.14159" />
+      <parent link="$(arg realsense_mount)"/>
+      <child link="realsense_mountpoint" />
     </joint>
-    <xacro:kinect_camera prefix="camera" robot_namespace="$(arg robot_namespace)"/>
+    <xacro:intel_realsense_mount prefix="camera" topic="realsense" parent_link="realsense_mountpoint"/>
   </xacro:if>
-  <!-- Velodyne Package. -->
-  <xacro:include filename="$(find velodyne_description)/urdf/HDL-32E.urdf.xacro"/>
-    <HDL-32E parent="base_link" name="velodyne" topic="/velodyne_points" hz=" 10" samples="220" gpu="${gpu}"> <!--Init Hz=10, sampling 220 -->
-    <origin xyz="0.25 0 0.55" rpy="0 0 0" />
-  </HDL-32E>
   <gazebo>
     <plugin name="gazebo_ros_control" filename="libgazebo_ros_control.so">
@@ -178,17 +181,4 @@
     </plugin>
   </gazebo>
-  <!-- Ground truth plugin. -->
-  <gazebo>
-  <plugin name="p3d_base_controller" filename="libgazebo_ros_p3d.so">
-    <alwaysOn>true</alwaysOn>
-    <updateRate>100.0</updateRate>
-    <bodyName>base_link</bodyName>
-    <topicName>ground_truth/odom</topicName>
-    <gaussianNoise>0.00</gaussianNoise>
-    <frameName>world</frameName>
-    <xyzOffsets>0 0 0</xyzOffsets>
-    <rpyOffsets>0 0 0</rpyOffsets>
-  </plugin>
-  </gazebo>
   <!-- Optional custom includes. -->
   <xacro:include filename="$(arg urdf_extras)" />

File: metro_sim/urdf/metro.urdf (robot description, URDF)
Before this commit: robot metro, 11 links, 10 joints
Joints:
- joint base_to_back_chassis: limit lower=-1.57 upper=1.57 effort=0.0 velocity=0.5 -> lower=-2.5 upper=2.5 effort=0.0 velocity=0.5
- joint base_to_bl_arm: limit lower=0 upper=0.65 effort=1000.0 velocity=0.5 -> lower=0 upper=0.60 effort=1000.0 velocity=0.5
- joint base_to_br_arm: axis 1 0 0 -> 0 1 0; limit lower=0 upper=0.65 effort=1000.0 velocity=0.5 -> lower=0 upper=0.6 effort=1000.0 velocity=0.5
- joint base_to_fl_arm: limit lower=0 upper=0.65 effort=1000.0 velocity=0.5 -> lower=-0.6 upper=0 effort=1000.0 velocity=0.5
- joint base_to_fr_arm: limit lower=0 upper=0.65 effort=1000.0 velocity=0.5 -> lower=-0.6 upper=0 effort=1000.0 velocity=0.5
